File: onewire.sch (KiCad schematic (older format))
At the start: 9 parts

Commit message: Update according to comments
Also add missing connectors and update the fuses
Parts:
- removed D?: BAT54S, Package_TO_SOT_SMD:SOT-23, symbol Diode:BAT54S
- removed FB?: GZ2012D601TF, symbol Device:Ferrite_Bead
- added U801: RCLAMP0524P-N, symbol SH-ESP32:RCLAMP0524P-N
- gave numbers to parts that had none: 7
Connections:
- net labels removed: Onewire_GND
- wire segments 12 -> 24
- no-connect marks 0 -> 4
Other:
- note removed: "FIXME: Is a BAT54S adequate for ESD\nprotection? is a clamping circuit even\nrequired?"
- moved on the sheet: C801, C802, C803, FB801, J801, R801, R802

Commit message: Rough PCB layout
Parts:
- C801: value 10u -> 10uF; footprint (none) -> Capacitor_SMD:C_0402_1005Metric
- C802: value 4700p -> 4.7nF/50V; footprint (none) -> Capacitor_SMD:C_0603_1608Metric
- C803: value 10u -> 10uF/50V; footprint (none) -> Capacitor_SMD:C_1206_3216Metric
- FB801: footprint (none) -> Inductor_SMD:L_0805_2012Metric
- J801: footprint (none) -> Connector_PinHeader_2.54mm:PinHeader_1x03_P2.54mm_Vertical
- R801: value 1.5k -> 2.2k; footprint (none) -> Resistor_SMD:R_0402_1005Metric
- R802: footprint (none) -> Resistor_SMD:R_0805_2012Metric
- U801: footprint (none) -> Package_DFN_QFN:Diodes_UDFN-10_1.0x2.5mm_P0.5mm
Connections:
- net +3V3: now also C801.1; no longer C803.1, U801.1 (IN1), U801.10 (OUT1)
- net Onewire_3V3: now also C803.1, U801.1 (IN1), U801.10 (OUT1); no longer C801.1
Other:
- moved on the sheet: C801, C803
Changed lines of the file:
@@
 AR Path="/5FAF30D4" Ref="R?"  Part="1"
 AR Path="/5FAEF03B/5FAF30D4" Ref="R801"  Part="1"
-F 0 "R801" V 4300 1550 50  0000 C CNN
-F 1 "1.5k" V 4300 1700 50  0000 C CNN
-F 2 "" V 4330 1600 50  0001 C CNN
+F 0 "R801" V 4200 1600 50  0000 C CNN
+F 1 "2.2k" V 4300 1600 50  0000 C CNN
+F 2 "Resistor_SMD:R_0402_1005Metric" V 4330 1600 50  0001 C CNN
 F 3 "~" H 4400 1600 50  0001 C CNN
 	1    4400 1600
@@
 F 0 "J801" H 1680 2492 50  0000 L CNN
 F 1 "Conn_01x03" H 1680 2401 50  0000 L CNN
-F 2 "" H 1600 2450 50  0001 C CNN
+F 2 "Connector_PinHeader_2.54mm:PinHeader_1x03_P2.54mm_Vertical" H 1600 2450 50  0001 C CNN
 F 3 "~" H 1600 2450 50  0001 C CNN
 	1    1600 2450
@@
 	0    1    -1   0
 $EndComp
-Wire Wire Line
-	5000 3900 4900 3900
-Wire Wire Line
-	4300 3900 4450 3900
 $Comp
 L Device:C C?
 U 1 1 5FAF4E24
-P 4900 4050
+P 4450 4050
 AR Path="/5FAF4E24" Ref="C?"  Part="1"
 AR Path="/5F9BE197/5FAF4E24" Ref="C?"  Part="1"
 AR Path="/5FAEF03B/5FAF4E24" Ref="C803"  Part="1"
-F 0 "C803" H 5015 4096 50  0000 L CNN
-F 1 "10u" H 5015 4005 50  0000 L CNN
-F 2 "" H 4938 3900 50  0001 C CNN
-F 3 "~" H 4900 4050 50  0001 C CNN
-	1    4900 4050
-	-1   0    0    -1
-$EndComp
-Connection ~ 4900 3900
-Wire Wire Line
-	4900 3900 4800 3900
+F 0 "C803" H 4565 4096 50  0000 L CNN
+F 1 "10uF/50V" H 4565 4005 50  0000 L CNN
+F 2 "Capacitor_SMD:C_1206_3216Metric" H 4488 3900 50  0001 C CNN
+F 3 "~" H 4450 4050 50  0001 C CNN
+	1    4450 4050
+	-1   0    0    -1
+$EndComp
 $Comp
 L power:GND #PWR?
 U 1 1 5FAF4E2C
-P 4900 4200
+P 4450 4200
 AR Path="/5FAF4E2C" Ref="#PWR?"  Part="1"
 AR Path="/5F9BE197/5FAF4E2C" Ref="#PWR?"  Part="1"
 AR Path="/5FAEF03B/5FAF4E2C" Ref="#PWR0808"  Part="1"
-F 0 "#PWR0808" H 4900 3950 50  0001 C CNN
-F 1 "GND" H 4905 4027 50  0000 C CNN
-F 2 "" H 4900 4200 50  0001 C CNN
-F 3 "" H 4900 4200 50  0001 C CNN
-	1    4900 4200
-	-1   0    0    -1
+F 0 "#PWR0808" H 4450 3950 50  0001 C CNN
+F 1 "GND" H 4455 4027 50  0000 C CNN
+F 2 "" H 4450 4200 50  0001 C CNN
+F 3 "" H 4450 4200 50  0001 C CNN
+	1    4450 4200
+	1    0    0    -1
 $EndComp
 $Comp
 L Device:C C?
 U 1 1 5FAF4E32
-P 4450 4050
+P 4850 4050
 AR Path="/5FAF4E32" Ref="C?"  Part="1"
 AR Path="/5F9BE197/5FAF4E32" Ref="C?"  Part="1"
 AR Path="/5FAEF03B/5FAF4E32" Ref="C801"  Part="1"
-F 0 "C801" H 4565 4096 50  0000 L CNN
-F 1 "10u" H 4565 4005 50  0000 L CNN
-F 2 "" H 4488 3900 50  0001 C CNN
-F 3 "~" H 4450 4050 50  0001 C CNN
-	1    4450 4050
-	-1   0    0    -1
-$EndComp
-Connection ~ 4450 3900
-Wire Wire Line
-	4450 3900 4500 3900
+F 0 "C801" H 4965 4096 50  0000 L CNN
+F 1 "10uF" H 4965 4005 50  0000 L CNN
+F 2 "Capacitor_SMD:C_0402_1005Metric" H 4888 3900 50  0001 C CNN
+F 3 "~" H 4850 4050 50  0001 C CNN
+	1    4850 4050
+	1    0    0    -1
+$EndComp
 $Comp
 L Device:Ferrite_Bead FB?
@@
 F 0 "FB801" V 4376 3900 50  0000 C CNN
 F 1 "GZ2012D601TF" V 4467 3900 50  0000 C CNN
-F 2 "" V 4580 3900 50  0001 C CNN
+F 2 "Inductor_SMD:L_0805_2012Metric" V 4580 3900 50  0001 C CNN
 F 3 "~" H 4650 3900 50  0001 C CNN
 	1    4650 3900
@@
 F 0 "R802" V 4193 2350 50  0000 C CNN
 F 1 "100R" V 4284 2350 50  0000 C CNN
-F 2 "" V 4330 2350 50  0001 C CNN
+F 2 "Resistor_SMD:R_0805_2012Metric" V 4330 2350 50  0001 C CNN
 F 3 "~" H 4400 2350 50  0001 C CNN
 	1    4400 2350
@@
 	1    0    0    -1
 $EndComp
-Text Notes 4500 1400 0    50   ~ 0
+Text Notes 4650 1400 0    50   ~ 0
 Pullup
 Text Notes 4600 2200 0    50   ~ 0
@@
 F 0 "U801" H 2450 4675 50  0000 C CNN
 F 1 "RCLAMP0524P-N" H 2450 4584 50  0000 C CNN
-F 2 "" H 2450 4150 50  0001 C CNN
+F 2 "Package_DFN_QFN:Diodes_UDFN-10_1.0x2.5mm_P0.5mm" H 2450 4150 50  0001 C CNN
 F 3 "" H 2450 4150 50  0001 C CNN
 	1    2450 4250
@@
 L power:GND #PWR?
 U 1 1 5FBFC117
-P 4450 4200
+P 4850 4200
 AR Path="/5FBFC117" Ref="#PWR?"  Part="1"
 AR Path="/5F9BE197/5FBFC117" Ref="#PWR?"  Part="1"
 AR Path="/5FAEF03B/5FBFC117" Ref="#PWR0806"  Part="1"
-F 0 "#PWR0806" H 4450 3950 50  0001 C CNN
-F 1 "GND" H 4455 4027 50  0000 C CNN
-F 2 "" H 4450 4200 50  0001 C CNN
-F 3 "" H 4450 4200 50  0001 C CNN
-	1    4450 4200
-	-1   0    0    -1
+F 0 "#PWR0806" H 4850 3950 50  0001 C CNN
+F 1 "GND" H 4855 4027 50  0000 C CNN
+F 2 "" H 4850 4200 50  0001 C CNN
+F 3 "" H 4850 4200 50  0001 C CNN
+	1    4850 4200
+	1    0    0    -1
 $EndComp
 Text Label 1650 3650 2    50   ~ 0
 DQ_CONN
-$Comp
-L power:+3.3V #PWR?
-U 1 1 5FBFC525
-P 1650 3750
-AR Path="/5FBFC525" Ref="#PWR?"  Part="1"
-AR Path="/5F9BE197/5FBFC525" Ref="#PWR?"  Part="1"
-AR Path="/5FAEF03B/5FBFC525" Ref="#PWR0801"  Part="1"
-F 0 "#PWR0801" H 1650 3600 50  0001 C CNN
-F 1 "+3.3V" V 1665 3878 50  0000 L CNN
-F 2 "" H 1650 3750 50  0001 C CNN
-F 3 "" H 1650 3750 50  0001 C CNN
-	1    1650 3750
-	0    -1   1    0
-$EndComp
 $Comp
 L power:GND #PWR?
@@
 P 4600 2550
 F 0 "C802" H 4715 2596 50  0000 L CNN
-F 1 "4700p" H 4715 2505 50  0000 L CNN
-F 2 "" H 4638 2400 50  0001 C CNN
+F 1 "4.7nF/50V" H 4715 2505 50  0000 L CNN
+F 2 "Capacitor_SMD:C_0603_1608Metric" H 4638 2400 50  0001 C CNN
 F 3 "~" H 4600 2550 50  0001 C CNN
 	1    4600 2550
 	1    0    0    -1
 $EndComp
+Wire Wire Line
+	4300 3900 4450 3900
+Connection ~ 4450 3900
+Wire Wire Line
+	4450 3900 4500 3900
+Wire Wire Line
+	4800 3900 4850 3900
+Connection ~ 4850 3900
+Wire Wire Line
+	4850 3900 5000 3900
+Text Label 1650 3750 2    50   ~ 0
+Onewire_3V3
 $EndSCHEMATC

Commit message: Specified JLCPCB footprints for components
Parts:
- C801: LCSC (none) -> C15525
- C802: LCSC (none) -> C53987
- C803: LCSC (none) -> C13585
- FB801: LCSC (none) -> C1017
- J801: LCSC (none) -> C358685
- R801: LCSC (none) -> C25879
- R802: LCSC (none) -> C17408
- U801: LCSC (none) -> C316044
Changed lines of the file:
@@
 F 2 "Resistor_SMD:R_0402_1005Metric" V 4330 1600 50  0001 C CNN
 F 3 "~" H 4400 1600 50  0001 C CNN
+F 4 "C25879" H 4400 1600 50  0001 C CNN "LCSC"
 	1    4400 1600
 	0    1    1    0
@@
 F 2 "Connector_PinHeader_2.54mm:PinHeader_1x03_P2.54mm_Vertical" H 1600 2450 50  0001 C CNN
 F 3 "~" H 1600 2450 50  0001 C CNN
+F 4 "C358685" H 1600 2450 50  0001 C CNN "LCSC"
 	1    1600 2450
 	-1   0    0    1
@@
 F 2 "Capacitor_SMD:C_1206_3216Metric" H 4488 3900 50  0001 C CNN
 F 3 "~" H 4450 4050 50  0001 C CNN
+F 4 "C13585" H 4450 4050 50  0001 C CNN "LCSC"
 	1    4450 4050
 	-1   0    0    -1
@@
 F 2 "Capacitor_SMD:C_0402_1005Metric" H 4888 3900 50  0001 C CNN
 F 3 "~" H 4850 4050 50  0001 C CNN
+F 4 "C15525" H 4850 4050 50  0001 C CNN "LCSC"
 	1    4850 4050
 	1    0    0    -1
@@
 F 2 "Inductor_SMD:L_0805_2012Metric" V 4580 3900 50  0001 C CNN
 F 3 "~" H 4650 3900 50  0001 C CNN
+F 4 "C1017" H 4650 3900 50  0001 C CNN "LCSC"
 	1    4650 3900
 	0    -1   1    0
@@
 F 2 "Resistor_SMD:R_0805_2012Metric" V 4330 2350 50  0001 C CNN
 F 3 "~" H 4400 2350 50  0001 C CNN
+F 4 "C17408" H 4400 2350 50  0001 C CNN "LCSC"
 	1    4400 2350
 	0    1    1    0
@@
 F 2 "Package_DFN_QFN:Diodes_UDFN-10_1.0x2.5mm_P0.5mm" H 2450 4150 50  0001 C CNN
 F 3 "" H 2450 4150 50  0001 C CNN
+F 4 "C316044" H 2450 4250 50  0001 C CNN "LCSC"
 	1    2450 4250
 	1    0    0    -1
@@
 F 2 "Capacitor_SMD:C_0603_1608Metric" H 4638 2400 50  0001 C CNN
 F 3 "~" H 4600 2550 50  0001 C CNN
+F 4 "C53987" H 4600 2550 50  0001 C CNN "LCSC"
 	1    4600 2550
 	1    0    0    -1
