File: optocouplers.sch (KiCad schematic (older format))
At the start: 19 parts

Commit message: Update according to comments
Also add missing connectors and update the fuses
Parts:
- removed J?: Screw_Terminal_01x04, symbol Connector:Screw_Terminal_01x04
- added D901: B5819W, symbol Device:D_Schottky
- added J901: Screw_Terminal_01x04, symbol Connector:Screw_Terminal_01x04
- gave numbers to parts that had none: 18
Connections:
- wire segments 40 -> 45
Other:
- note added: "A relay can be connected between\nV_ISO_CONN and ISO_OUT_CONN"
- note removed: "FIXME: What do we want to achieve with\nthe optoisolated output? Could also\nmake a relay driver"
- moved on the sheet: C901, C902, C903, C904, C905, C906, FB901, FB902, FB903, FB904, Q901, R901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

Commit message: Rough PCB layout
Parts:
- removed FB901: GZ2012D601TF, symbol Device:Ferrite_Bead
- removed J901: Screw_Terminal_01x04, symbol Connector:Screw_Terminal_01x04
- added J901: Conn_01x04, Connector_PinHeader_2.54mm:PinHeader_1x04_P2.54mm_Vertical, symbol Connector_Generic:Conn_01x04
- C901: value 10u -> 10uF; footprint (none) -> Capacitor_SMD:C_0402_1005Metric
- C902, C903: value 33p -> 33pF; footprint (none) -> Capacitor_SMD:C_0402_1005Metric
- C904: value 10u -> 10uF/50V; footprint (none) -> Capacitor_SMD:C_1206_3216Metric
- C905, C906: value 33p -> 33pF/50V; footprint (none) -> Capacitor_SMD:C_0603_1608Metric
- D901: footprint (none) -> Diode_SMD:D_SOD-123
- FB902, FB903, FB904: footprint (none) -> Inductor_SMD:L_0805_2012Metric
- R901, R905: footprint (none) -> Resistor_SMD:R_0603_1608Metric
- R902, R903, R904: footprint (none) -> Resistor_SMD:R_0402_1005Metric
- U901, U902: value EL817 -> EL817S1; footprint Package_DIP:DIP-4_W7.62mm -> Package_SO:SSO-4_6.7x5.1mm_P2.54mm_Clearance8mm
Connections:
- net labels removed: ISO_GND_CONN
- wire segments 45 -> 43
Changed lines of the file:
@@
 F 0 "R901" V 2143 4300 50  0000 C CNN
 F 1 "220R" V 2234 4300 50  0000 C CNN
-F 2 "" V 2280 4300 50  0001 C CNN
+F 2 "Resistor_SMD:R_0603_1608Metric" V 2280 4300 50  0001 C CNN
 F 3 "~" H 2350 4300 50  0001 C CNN
 	1    2350 4300
@@
 P 2900 4400
 F 0 "U901" H 2900 4725 50  0000 C CNN
-F 1 "EL817" H 2900 4634 50  0000 C CNN
-F 2 "Package_DIP:DIP-4_W7.62mm" H 2700 4200 50  0001 L CIN
+F 1 "EL817S1" H 2900 4634 50  0000 C CNN
+F 2 "Package_SO:SSO-4_6.7x5.1mm_P2.54mm_Clearance8mm" H 2700 4200 50  0001 L CIN
 F 3 "http://www.everlight.com/file/ProductFile/EL817.pdf" H 2900 4400 50  0001 L CNN
 	1    2900 4400
@@
 F 0 "R903" H 3420 3946 50  0000 L CNN
 F 1 "5.1k" H 3420 3855 50  0000 L CNN
-F 2 "" V 3280 3900 50  0001 C CNN
+F 2 "Resistor_SMD:R_0402_1005Metric" V 3280 3900 50  0001 C CNN
 F 3 "~" H 3350 3900 50  0001 C CNN
 	1    3350 3900
@@
 F 0 "R904" H 3970 3846 50  0000 L CNN
 F 1 "5.1k" H 3970 3755 50  0000 L CNN
-F 2 "" V 3830 3800 50  0001 C CNN
+F 2 "Resistor_SMD:R_0402_1005Metric" V 3830 3800 50  0001 C CNN
 F 3 "~" H 3900 3800 50  0001 C CNN
 	1    3900 3800
@@
 P 3400 2400
 F 0 "U902" H 3400 2725 50  0000 C CNN
-F 1 "EL817" H 3400 2634 50  0000 C CNN
-F 2 "Package_DIP:DIP-4_W7.62mm" H 3200 2200 50  0001 L CIN
+F 1 "EL817S1" H 3400 2634 50  0000 C CNN
+F 2 "Package_SO:SSO-4_6.7x5.1mm_P2.54mm_Clearance8mm" H 3200 2200 50  0001 L CIN
 F 3 "http://www.everlight.com/file/ProductFile/EL817.pdf" H 3400 2400 50  0001 L CNN
 	1    3400 2400
@@
 F 0 "R905" V 3743 2300 50  0000 C CNN
 F 1 "1k" V 3834 2300 50  0000 C CNN
-F 2 "" V 3880 2300 50  0001 C CNN
+F 2 "Resistor_SMD:R_0603_1608Metric" V 3880 2300 50  0001 C CNN
 F 3 "~" H 3950 2300 50  0001 C CNN
 	1    3950 2300
@@
 F 0 "R902" H 2920 1996 50  0000 L CNN
 F 1 "5.1k" H 2920 1905 50  0000 L CNN
-F 2 "" V 2780 1950 50  0001 C CNN
+F 2 "Resistor_SMD:R_0402_1005Metric" V 2780 1950 50  0001 C CNN
 F 3 "~" H 2850 1950 50  0001 C CNN
 	1    2850 1950
@@
 F 0 "FB902" V 6776 1700 50  0000 C CNN
 F 1 "GZ2012D601TF" V 6867 1700 50  0000 C CNN
-F 2 "" V 6980 1700 50  0001 C CNN
+F 2 "Inductor_SMD:L_0805_2012Metric" V 6980 1700 50  0001 C CNN
 F 3 "~" H 7050 1700 50  0001 C CNN
 	1    7050 1700
-	0    1    1    0
-$EndComp
-$Comp
-L Device:Ferrite_Bead FB?
-U 1 1 5FB45373
-P 7050 1200
-AR Path="/5F89C30A/5FB45373" Ref="FB?"  Part="1"
-AR Path="/5FB2AE13/5FB45373" Ref="FB901"  Part="1"
-F 0 "FB901" V 6776 1200 50  0000 C CNN
-F 1 "GZ2012D601TF" V 6867 1200 50  0000 C CNN
-F 2 "" V 6980 1200 50  0001 C CNN
-F 3 "~" H 7050 1200 50  0001 C CNN
-	1    7050 1200
 	0    1    1    0
 $EndComp
@@
 AR Path="/5FB2AE13/5FB49AD1" Ref="C902"  Part="1"
 F 0 "C902" H 6965 3146 50  0000 L CNN
-F 1 "33p" H 6965 3055 50  0000 L CNN
-F 2 "" H 6888 2950 50  0001 C CNN
+F 1 "33pF" H 6965 3055 50  0000 L CNN
+F 2 "Capacitor_SMD:C_0402_1005Metric" H 6888 2950 50  0001 C CNN
 F 3 "~" H 6850 3100 50  0001 C CNN
 	1    6850 3100
-	1    0    0    -1
+	-1   0    0    -1
 $EndComp
 $Comp
@@
 AR Path="/5FB2AE13/5FB49ADD" Ref="C905"  Part="1"
 F 0 "C905" H 7415 3146 50  0000 L CNN
-F 1 "33p" H 7415 3055 50  0000 L CNN
-F 2 "" H 7338 2950 50  0001 C CNN
+F 1 "33pF/50V" H 7415 3055 50  0000 L CNN
+F 2 "Capacitor_SMD:C_0603_1608Metric" H 7338 2950 50  0001 C CNN
 F 3 "~" H 7300 3100 50  0001 C CNN
 	1    7300 3100
@@
 F 0 "FB903" V 6826 2950 50  0000 C CNN
 F 1 "GZ2012D101TF" V 6917 2950 50  0000 C CNN
-F 2 "" V 7030 2950 50  0001 C CNN
+F 2 "Inductor_SMD:L_0805_2012Metric" V 7030 2950 50  0001 C CNN
 F 3 "~" H 7100 2950 50  0001 C CNN
 	1    7100 2950
 	0    1    1    0
 $EndComp
-Wire Wire Line
-	7350 1200 7200 1200
 Wire Wire Line
 	7300 1700 7200 1700
@@
 ISO_IN
 Text Label 9350 2700 2    50   ~ 0
-ISO_GND_CONN
+ISO_GND
 Text Label 9350 2800 2    50   ~ 0
 V_ISO_CONN
@@
 Text Label 9350 3000 2    50   ~ 0
 ISO_OUT_CONN
-Text Label 7350 1200 0    50   ~ 0
-ISO_GND_CONN
-Text Label 6700 1200 2    50   ~ 0
-ISO_GND
-Wire Wire Line
-	6900 1200 6700 1200
 $Comp
 L Device:C C?
@@
 AR Path="/5FB2AE13/5FB5449D" Ref="C904"  Part="1"
 F 0 "C904" H 7415 1896 50  0000 L CNN
-F 1 "10u" H 7415 1805 50  0000 L CNN
-F 2 "" H 7338 1700 50  0001 C CNN
+F 1 "10uF/50V" H 7415 1805 50  0000 L CNN
+F 2 "Capacitor_SMD:C_1206_3216Metric" H 7338 1700 50  0001 C CNN
 F 3 "~" H 7300 1850 50  0001 C CNN
 	1    7300 1850
-	-1   0    0    -1
+	1    0    0    -1
 $EndComp
 $Comp
@@
 AR Path="/5FB2AE13/5FB54A5E" Ref="C901"  Part="1"
 F 0 "C901" H 6915 1896 50  0000 L CNN
-F 1 "10u" H 6915 1805 50  0000 L CNN
-F 2 "" H 6838 1700 50  0001 C CNN
+F 1 "10uF" H 6915 1805 50  0000 L CNN
+F 2 "Capacitor_SMD:C_0402_1005Metric" H 6838 1700 50  0001 C CNN
 F 3 "~" H 6800 1850 50  0001 C CNN
 	1    6800 1850
@@
 Connection ~ 6800 1700
 Text Label 7300 2000 3    50   ~ 0
-ISO_GND_CONN
+ISO_GND
 Text Label 6800 2000 3    50   ~ 0
 ISO_GND
@@
 V_ISO_CONN
 Text Label 7300 3250 3    50   ~ 0
-ISO_GND_CONN
+ISO_GND
 Text Label 7450 4100 0    50   ~ 0
 ISO_OUT_CONN
@@
 AR Path="/5FB2AE13/5FB5DCAF" Ref="C903"  Part="1"
 F 0 "C903" H 6965 4296 50  0000 L CNN
-F 1 "33p" H 6965 4205 50  0000 L CNN
-F 2 "" H 6888 4100 50  0001 C CNN
+F 1 "33pF" H 6965 4205 50  0000 L CNN
+F 2 "Capacitor_SMD:C_0402_1005Metric" H 6888 4100 50  0001 C CNN
 F 3 "~" H 6850 4250 50  0001 C CNN
 	1    6850 4250
-	1    0    0    -1
+	-1   0    0    -1
 $EndComp
 $Comp
@@
 AR Path="/5FB2AE13/5FB5DCB5" Ref="C906"  Part="1"
 F 0 "C906" H 7415 4296 50  0000 L CNN
-F 1 "33p" H 7415 4205 50  0000 L CNN
-F 2 "" H 7338 4100 50  0001 C CNN
+F 1 "33pF/50V" H 7415 4205 50  0000 L CNN
+F 2 "Capacitor_SMD:C_0603_1608Metric" H 7338 4100 50  0001 C CNN
 F 3 "~" H 7300 4250 50  0001 C CNN
 	1    7300 4250
@@
 F 0 "FB904" V 6826 4100 50  0000 C CNN
 F 1 "GZ2012D101TF" V 6917 4100 50  0000 C CNN
-F 2 "" V 7030 4100 50  0001 C CNN
+F 2 "Inductor_SMD:L_0805_2012Metric" V 7030 4100 50  0001 C CNN
 F 3 "~" H 7100 4100 50  0001 C CNN
 	1    7100 4100
@@
 ISO_OUT
 Text Label 7300 4400 3    50   ~ 0
-ISO_GND_CONN
+ISO_GND
 Wire Wire Line
 	3900 4000 4250 4000
@@
 F 0 "D901" V 4204 3879 50  0000 L CNN
 F 1 "B5819W" V 4295 3879 50  0000 L CNN
-F 2 "" H 4250 3800 50  0001 C CNN
+F 2 "Diode_SMD:D_SOD-123" H 4250 3800 50  0001 C CNN
 F 3 "~" H 4250 3800 50  0001 C CNN
 F 4 "" V 4250 3800 50  0001 C CNN "Notes"
@@
 	3900 3600 3900 3500
 $Comp
-L Connector:Screw_Terminal_01x04 J901
-U 1 1 5FC6C76D
+L Connector_Generic:Conn_01x04 J901
+U 1 1 5F95832D
 P 9550 2800
 F 0 "J901" H 9630 2792 50  0000 L CNN
-F 1 "Screw_Terminal_01x04" H 9630 2701 50  0000 L CNN
-F 2 "" H 9550 2800 50  0001 C CNN
+F 1 "Conn_01x04" H 9630 2701 50  0000 L CNN
+F 2 "Connector_PinHeader_2.54mm:PinHeader_1x04_P2.54mm_Vertical" H 9550 2800 50  0001 C CNN
 F 3 "~" H 9550 2800 50  0001 C CNN
 	1    9550 2800

Commit message: Specified JLCPCB footprints for components
Parts:
- C901: LCSC (none) -> C15525
- C902, C903: LCSC (none) -> C1562
- C904: LCSC (none) -> C13585
- C905, C906: LCSC (none) -> C1663
- FB902: LCSC (none) -> C1017
- FB903, FB904: LCSC (none) -> C1015
- J901: LCSC (none) -> C358686
- Q901: LCSC (none) -> C41095
- R901: LCSC (none) -> C22962
- R902, R903, R904: LCSC (none) -> C25905
- R905: LCSC (none) -> C21190
- U901, U902: LCSC (none) -> C106900
Changed lines of the file:
@@
 F 2 "Resistor_SMD:R_0603_1608Metric" V 2280 4300 50  0001 C CNN
 F 3 "~" H 2350 4300 50  0001 C CNN
+F 4 "C22962" H 2350 4300 50  0001 C CNN "LCSC"
 	1    2350 4300
 	0    1    1    0
@@
 F 2 "Package_SO:SSO-4_6.7x5.1mm_P2.54mm_Clearance8mm" H 2700 4200 50  0001 L CIN
 F 3 "http://www.everlight.com/file/ProductFile/EL817.pdf" H 2900 4400 50  0001 L CNN
+F 4 "C106900" H 2900 4400 50  0001 C CNN "LCSC"
 	1    2900 4400
 	1    0    0    -1
@@
 F 2 "Package_TO_SOT_SMD:SOT-23" H 4000 4225 50  0001 L CIN
 F 3 "www.onsemi.com/pub/Collateral/MMBT5550LT1-D.PDF" H 3800 4300 50  0001 L CNN
+F 4 "C41095" H 3800 4300 50  0001 C CNN "LCSC"
 	1    3800 4300
 	1    0    0    -1
@@
 F 2 "Resistor_SMD:R_0402_1005Metric" V 3280 3900 50  0001 C CNN
 F 3 "~" H 3350 3900 50  0001 C CNN
+F 4 "C25905" H 3350 3900 50  0001 C CNN "LCSC"
 	1    3350 3900
 	1    0    0    -1
@@
 F 2 "Resistor_SMD:R_0402_1005Metric" V 3830 3800 50  0001 C CNN
 F 3 "~" H 3900 3800 50  0001 C CNN
+F 4 "C25905" H 3900 3800 50  0001 C CNN "LCSC"
 	1    3900 3800
 	1    0    0    -1
@@
 F 2 "Package_SO:SSO-4_6.7x5.1mm_P2.54mm_Clearance8mm" H 3200 2200 50  0001 L CIN
 F 3 "http://www.everlight.com/file/ProductFile/EL817.pdf" H 3400 2400 50  0001 L CNN
+F 4 "C106900" H 3400 2400 50  0001 C CNN "LCSC"
 	1    3400 2400
 	-1   0    0    -1
@@
 F 2 "Resistor_SMD:R_0603_1608Metric" V 3880 2300 50  0001 C CNN
 F 3 "~" H 3950 2300 50  0001 C CNN
+F 4 "C21190" H 3950 2300 50  0001 C CNN "LCSC"
 	1    3950 2300
 	0    1    1    0
@@
 F 2 "Resistor_SMD:R_0402_1005Metric" V 2780 1950 50  0001 C CNN
 F 3 "~" H 2850 1950 50  0001 C CNN
+F 4 "C25905" H 2850 1950 50  0001 C CNN "LCSC"
 	1    2850 1950
 	1    0    0    -1
@@
 F 2 "Inductor_SMD:L_0805_2012Metric" V 6980 1700 50  0001 C CNN
 F 3 "~" H 7050 1700 50  0001 C CNN
+F 4 "C1017" H 7050 1700 50  0001 C CNN "LCSC"
 	1    7050 1700
 	0    1    1    0
@@
 F 2 "Capacitor_SMD:C_0402_1005Metric" H 6888 2950 50  0001 C CNN
 F 3 "~" H 6850 3100 50  0001 C CNN
+F 4 "C1562" H 6850 3100 50  0001 C CNN "LCSC"
 	1    6850 3100
 	-1   0    0    -1
@@
 F 2 "Capacitor_SMD:C_0603_1608Metric" H 7338 2950 50  0001 C CNN
 F 3 "~" H 7300 3100 50  0001 C CNN
+F 4 "C1663" H 7300 3100 50  0001 C CNN "LCSC"
 	1    7300 3100
 	1    0    0    -1
@@
 F 2 "Inductor_SMD:L_0805_2012Metric" V 7030 2950 50  0001 C CNN
 F 3 "~" H 7100 2950 50  0001 C CNN
+F 4 "C1015" H 7100 2950 50  0001 C CNN "LCSC"
 	1    7100 2950
 	0    1    1    0
@@
 F 2 "Capacitor_SMD:C_1206_3216Metric" H 7338 1700 50  0001 C CNN
 F 3 "~" H 7300 1850 50  0001 C CNN
+F 4 "C13585" H 7300 1850 50  0001 C CNN "LCSC"
 	1    7300 1850
 	1    0    0    -1
@@
 F 2 "Capacitor_SMD:C_0402_1005Metric" H 6838 1700 50  0001 C CNN
 F 3 "~" H 6800 1850 50  0001 C CNN
+F 4 "C15525" H 6800 1850 50  0001 C CNN "LCSC"
 	1    6800 1850
 	-1   0    0    -1
@@
 F 2 "Capacitor_SMD:C_0402_1005Metric" H 6888 4100 50  0001 C CNN
 F 3 "~" H 6850 4250 50  0001 C CNN
+F 4 "C1562" H 6850 4250 50  0001 C CNN "LCSC"
 	1    6850 4250
 	-1   0    0    -1
@@
 F 2 "Capacitor_SMD:C_0603_1608Metric" H 7338 4100 50  0001 C CNN
 F 3 "~" H 7300 4250 50  0001 C CNN
+F 4 "C1663" H 7300 4250 50  0001 C CNN "LCSC"
 	1    7300 4250
 	1    0    0    -1
@@
 F 2 "Inductor_SMD:L_0805_2012Metric" V 7030 4100 50  0001 C CNN
 F 3 "~" H 7100 4100 50  0001 C CNN
+F 4 "C1015" H 7100 4100 50  0001 C CNN "LCSC"
 	1    7100 4100
 	0    1    1    0
@@
 F 2 "Connector_PinHeader_2.54mm:PinHeader_1x04_P2.54mm_Vertical" H 9550 2800 50  0001 C CNN
 F 3 "~" H 9550 2800 50  0001 C CNN
+F 4 "C358686" H 9550 2800 50  0001 C CNN "LCSC"
 	1    9550 2800
 	1    0    0    -1

Commit message: Change optocoupler types, improve ground planes and a lot of other smaller fixes
Parts:
- removed U901, U902: EL817S1, Package_SO:SSO-4_6.7x5.1mm_P2.54mm_Clearance8mm, symbol Isolator:EL817
- added D902: SM4007PL, Diode_SMD:D_SOD-123F, symbol Device:D
- added U901, U902: EL3H7(C)(TA)-G, Package_SO:SOP-4_4.4x2.6mm_P1.27mm, symbol SH-ESP32:EL3H7
- D901: value B5819W -> SM4007PL; footprint Diode_SMD:D_SOD-123 -> Diode_SMD:D_SOD-123F; symbol Device:D_Schottky -> Device:D; LCSC C8598 -> C64898
- R902: value 5.1k -> 2.2k; footprint Resistor_SMD:R_0402_1005Metric -> Resistor_SMD:R_0603_1608Metric; LCSC C25905 -> C4190
- R903, R904: value 5.1k -> 3.9k; footprint Resistor_SMD:R_0402_1005Metric -> Resistor_SMD:R_0603_1608Metric; LCSC C25905 -> C23018
- R905: value 1k -> 3.9k; LCSC C21190 -> C23018
Connections:
- wire segments 43 -> 46
Other:
- note added: "Design criteria: ISO_IN voltage swinging \nfrom roughly 0.6V to 4.2V causes \nIN1 to swing from 0V to 3.3V,\nabsolute maximum input voltage 18V."
- note added: "Diode for reverse polarity protection"
- note added: "Flyback diode for inductive loads"
- note added: "ISO_OUT switches from 0 to V_ISO\nas OUT1 rises above 1.2V."
- moved on the sheet: R902, R905
Changed lines of the file:
@@
 	2200 4300 2100 4300
-$Comp
-L Isolator:EL817 U901
-U 1 1 5FB321C6
-P 2900 4400
-F 0 "U901" H 2900 4725 50  0000 C CNN
-F 1 "EL817S1" H 2900 4634 50  0000 C CNN
-F 2 "Package_SO:SSO-4_6.7x5.1mm_P2.54mm_Clearance8mm" H 2700 4200 50  0001 L CIN
-F 3 "http://www.everlight.com/file/ProductFile/EL817.pdf" H 2900 4400 50  0001 L CNN
-F 4 "C106900" H 2900 4400 50  0001 C CNN "LCSC"
-	1    2900 4400
-	1    0    0    -1
-$EndComp
 $Comp
 L Transistor_BJT:MMBT5551L Q901
@@
 P 3350 3900
 F 0 "R903" H 3420 3946 50  0000 L CNN
-F 1 "5.1k" H 3420 3855 50  0000 L CNN
-F 2 "Resistor_SMD:R_0402_1005Metric" V 3280 3900 50  0001 C CNN
+F 1 "3.9k" H 3420 3855 50  0000 L CNN
+F 2 "Resistor_SMD:R_0603_1608Metric" V 3280 3900 50  0001 C CNN
 F 3 "~" H 3350 3900 50  0001 C CNN
-F 4 "C25905" H 3350 3900 50  0001 C CNN "LCSC"
+F 4 "C23018" H 3350 3900 50  0001 C CNN "LCSC"
 	1    3350 3900
 	1    0    0    -1
@@
 P 3900 3800
 F 0 "R904" H 3970 3846 50  0000 L CNN
-F 1 "5.1k" H 3970 3755 50  0000 L CNN
-F 2 "Resistor_SMD:R_0402_1005Metric" V 3830 3800 50  0001 C CNN
+F 1 "3.9k" H 3970 3755 50  0000 L CNN
+F 2 "Resistor_SMD:R_0603_1608Metric" V 3830 3800 50  0001 C CNN
 F 3 "~" H 3900 3800 50  0001 C CNN
-F 4 "C25905" H 3900 3800 50  0001 C CNN "LCSC"
+F 4 "C23018" H 3900 3800 50  0001 C CNN "LCSC"
 	1    3900 3800
 	1    0    0    -1
@@
 	3900 4500 3900 4750
 Wire Wire Line
-	3300 4750 3300 4500
+	3300 4950 3300 4500
 Wire Wire Line
 	3300 4500 3200 4500
-Wire Wire Line
-	3300 4750 3600 4750
-Wire Wire Line
-	3600 4750 3600 4900
-Connection ~ 3600 4750
-Wire Wire Line
-	3600 4750 3900 4750
-Text Label 3600 4900 3    50   ~ 0
+Text Label 3900 4750 3    50   ~ 0
 ISO_GND
 Text Label 4800 4000 0    50   ~ 0
@@
 Text Label 3900 3500 1    50   ~ 0
 V_ISO
-$Comp
-L Isolator:EL817 U902
-U 1 1 5FB3BE11
-P 3400 2400
-F 0 "U902" H 3400 2725 50  0000 C CNN
-F 1 "EL817S1" H 3400 2634 50  0000 C CNN
-F 2 "Package_SO:SSO-4_6.7x5.1mm_P2.54mm_Clearance8mm" H 3200 2200 50  0001 L CIN
-F 3 "http://www.everlight.com/file/ProductFile/EL817.pdf" H 3400 2400 50  0001 L CNN
-F 4 "C106900" H 3400 2400 50  0001 C CNN "LCSC"
-	1    3400 2400
-	-1   0    0    -1
-$EndComp
-Text Label 3900 2700 3    50   ~ 0
-ISO_GND
-$Comp
-L Device:R R905
-U 1 1 5FB3CD58
-P 3950 2300
-F 0 "R905" V 3743 2300 50  0000 C CNN
-F 1 "1k" V 3834 2300 50  0000 C CNN
-F 2 "Resistor_SMD:R_0603_1608Metric" V 3880 2300 50  0001 C CNN
-F 3 "~" H 3950 2300 50  0001 C CNN
-F 4 "C21190" H 3950 2300 50  0001 C CNN "LCSC"
-	1    3950 2300
-	0    1    1    0
-$EndComp
+Text Label 4700 2750 0    50   ~ 0
+ISO_GND
 $Comp
 L Device:R R902
 U 1 1 5FB3D3D9
-P 2850 1950
-F 0 "R902" H 2920 1996 50  0000 L CNN
-F 1 "5.1k" H 2920 1905 50  0000 L CNN
-F 2 "Resistor_SMD:R_0402_1005Metric" V 2780 1950 50  0001 C CNN
-F 3 "~" H 2850 1950 50  0001 C CNN
-F 4 "C25905" H 2850 1950 50  0001 C CNN "LCSC"
-	1    2850 1950
+P 2850 2700
+F 0 "R902" H 2920 2746 50  0000 L CNN
+F 1 "2.2k" H 2920 2655 50  0000 L CNN
+F 2 "Resistor_SMD:R_0603_1608Metric" V 2780 2700 50  0001 C CNN
+F 3 "~" H 2850 2700 50  0001 C CNN
+F 4 "C4190" H 2850 2700 50  0001 C CNN "LCSC"
+	1    2850 2700
 	1    0    0    -1
 $EndComp
@@
 L power:+3.3V #PWR0903
 U 1 1 5FB3DDF1
-P 2850 1800
-F 0 "#PWR0903" H 2850 1650 50  0001 C CNN
-F 1 "+3.3V" H 2865 1973 50  0000 C CNN
-F 2 "" H 2850 1800 50  0001 C CNN
-F 3 "" H 2850 1800 50  0001 C CNN
-	1    2850 1800
+P 2850 2100
+F 0 "#PWR0903" H 2850 1950 50  0001 C CNN
+F 1 "+3.3V" H 2865 2273 50  0000 C CNN
+F 2 "" H 2850 2100 50  0001 C CNN
+F 3 "" H 2850 2100 50  0001 C CNN
+	1    2850 2100
 	1    0    0    -1
 $EndComp
@@
 L power:GND #PWR0902
 U 1 1 5FB3E620
-P 2750 2700
-F 0 "#PWR0902" H 2750 2450 50  0001 C CNN
-F 1 "GND" H 2755 2527 50  0000 C CNN
-F 2 "" H 2750 2700 50  0001 C CNN
-F 3 "" H 2750 2700 50  0001 C CNN
-	1    2750 2700
-	1    0    0    -1
-$EndComp
-Wire Wire Line
-	2750 2700 2750 2500
-Wire Wire Line
-	2750 2500 3100 2500
+P 2850 2950
+F 0 "#PWR0902" H 2850 2700 50  0001 C CNN
+F 1 "GND" H 2855 2777 50  0000 C CNN
+F 2 "" H 2850 2950 50  0001 C CNN
+F 3 "" H 2850 2950 50  0001 C CNN
+	1    2850 2950
+	1    0    0    -1
+$EndComp
+Wire Wire Line
+	2850 2950 2850 2850
+Wire Wire Line
+	2850 2500 3100 2500
 Wire Wire Line
 	3100 2300 2850 2300
@@
 	2850 2300 2850 2100
 Wire Wire Line
-	2850 2300 2600 2300
-Connection ~ 2850 2300
-Wire Wire Line
-	3700 2500 3900 2500
-Wire Wire Line
-	3900 2500 3900 2700
-Wire Wire Line
-	3800 2300 3700 2300
-Wire Wire Line
-	4100 2300 4250 2300
-Text Label 4250 2300 0    50   ~ 0
+	2850 2500 2600 2500
+Text Label 4700 2300 0    50   ~ 0
 ISO_IN
 $Comp
@@
 Wire Wire Line
 	3900 4000 4250 4000
-Text HLabel 2600 2300 0    50   Input ~ 0
+Text HLabel 2600 2500 0    50   Input ~ 0
 IN1
 Text HLabel 2100 4300 0    50   Input ~ 0
 OUT1
 $Comp
-L Device:D_Schottky D?
+L Device:D D?
 U 1 1 5FC24243
 P 4250 3800
@@
 AR Path="/5FB2AE13/5FC24243" Ref="D901"  Part="1"
 F 0 "D901" V 4204 3879 50  0000 L CNN
-F 1 "B5819W" V 4295 3879 50  0000 L CNN
-F 2 "Diode_SMD:D_SOD-123" H 4250 3800 50  0001 C CNN
+F 1 "SM4007PL" V 4295 3879 50  0000 L CNN
+F 2 "Diode_SMD:D_SOD-123F" H 4250 3800 50  0001 C CNN
 F 3 "~" H 4250 3800 50  0001 C CNN
 F 4 "" V 4250 3800 50  0001 C CNN "Notes"
-F 5 "C8598" H 4250 3800 50  0001 C CNN "LCSC"
+F 5 "C64898" H 4250 3800 50  0001 C CNN "LCSC"
 	1    4250 3800
 	0    1    1    0
@@
 	1    0    0    -1
 $EndComp
+Text Notes 3400 1850 0    50   ~ 0
+Design criteria: ISO_IN voltage swinging \nfrom roughly 0.6V to 4.2V causes \nIN1 to swing from 0V to 3.3V,\nabsolute maximum input voltage 18V.
+Text Notes 4150 5050 0    50   ~ 0
+ISO_OUT switches from 0 to V_ISO\nas OUT1 rises above 1.2V.
+Text Label 3300 4750 3    50   ~ 0
+ISO_GND
+Wire Wire Line
+	4550 2300 4700 2300
+Wire Wire Line
+	4250 2300 4100 2300
+$Comp
+L Device:R R905
+U 1 1 5FB3CD58
+P 4400 2300
+F 0 "R905" V 4193 2300 50  0000 C CNN
+F 1 "3.9k" V 4284 2300 50  0000 C CNN
+F 2 "Resistor_SMD:R_0603_1608Metric" V 4330 2300 50  0001 C CNN
+F 3 "~" H 4400 2300 50  0001 C CNN
+F 4 "C23018" H 4400 2300 50  0001 C CNN "LCSC"
+	1    4400 2300
+	0    1    1    0
+$EndComp
+Wire Wire Line
+	2850 2550 2850 2500
+Connection ~ 2850 2500
+$Comp
+L Device:D D?
+U 1 1 5FC9D466
+P 4100 2500
+AR Path="/5C348474/5FC9D466" Ref="D?"  Part="1"
+AR Path="/5E460E30/5FC9D466" Ref="D?"  Part="1"
+AR Path="/5F6FAF6E/5FC9D466" Ref="D?"  Part="1"
+AR Path="/5F733BA4/5FC9D466" Ref="D?"  Part="1"
+AR Path="/5FB2AE13/5FC9D466" Ref="D902"  Part="1"
+F 0 "D902" V 4050 2650 50  0000 C CNN
+F 1 "SM4007PL" V 4150 2750 50  0000 C CNN
+F 2 "Diode_SMD:D_SOD-123F" H 4100 2500 50  0001 C CNN
+F 3 "~" H 4100 2500 50  0001 C CNN
+F 4 "C64898" H 4100 2500 50  0001 C CNN "LCSC"
+	1    4100 2500
+	0    1    1    0
+$EndComp
+Wire Wire Line
+	3700 2500 3900 2500
+Wire Wire Line
+	3900 2500 3900 2750
+Wire Wire Line
+	3900 2750 4100 2750
+Wire Wire Line
+	4100 2350 4100 2300
+Connection ~ 4100 2300
+Wire Wire Line
+	4100 2300 3700 2300
+Wire Wire Line
+	4100 2650 4100 2750
+Connection ~ 4100 2750
+Wire Wire Line
+	4100 2750 4700 2750
+Text Notes 4700 2550 0    50   ~ 0
+Diode for reverse polarity protection
+Text Notes 4800 3800 0    50   ~ 0
+Flyback diode for inductive loads
+$Comp
+L SH-ESP32:EL3H7 U902
+U 1 1 5FCA98FD
+P 3400 2400
+F 0 "U902" H 3400 2725 50  0000 C CNN
+F 1 "EL3H7(C)(TA)-G" H 3400 2634 50  0000 C CNN
+F 2 "Package_SO:SOP-4_4.4x2.6mm_P1.27mm" H 3200 2200 50  0001 L CIN
+F 3 "http://www.sharpsme.com/download/pc3h4-epdf" H 3425 2400 50  0001 L CNN
+	1    3400 2400
+	-1   0    0    -1
+$EndComp
+$Comp
+L SH-ESP32:EL3H7 U901
+U 1 1 5FCB38F6
+P 2900 4400
+F 0 "U901" H 2900 4725 50  0000 C CNN
+F 1 "EL3H7(C)(TA)-G" H 2900 4634 50  0000 C CNN
+F 2 "Package_SO:SOP-4_4.4x2.6mm_P1.27mm" H 2700 4200 50  0001 L CIN
+F 3 "http://www.sharpsme.com/download/pc3h4-epdf" H 2925 4400 50  0001 L CNN
+	1    2900 4400
+	1    0    0    -1
+$EndComp

Commit message: Add a missing LCSC part number for U901 and U902
Parts:
- U901, U902: LCSC (none) -> C92243
Changed lines of the file:
@@
 F 2 "Package_SO:SOP-4_4.4x2.6mm_P1.27mm" H 3200 2200 50  0001 L CIN
 F 3 "http://www.sharpsme.com/download/pc3h4-epdf" H 3425 2400 50  0001 L CNN
+F 4 "C92243" H 3400 2400 50  0001 C CNN "LCSC"
 	1    3400 2400
 	-1   0    0    -1
@@
 F 2 "Package_SO:SOP-4_4.4x2.6mm_P1.27mm" H 2700 4200 50  0001 L CIN
 F 3 "http://www.sharpsme.com/download/pc3h4-epdf" H 2925 4400 50  0001 L CNN
+F 4 "C92243" H 2900 4400 50  0001 C CNN "LCSC"
 	1    2900 4400
 	1    0    0    -1
