File: optocouplers.sch (KiCad schematic (older format))
At the start: 21 parts, among them J901 Conn_01x04, Q901 MMBT5551L, U901 EL3H7(C)(TA)-G, U902 EL3H7(C)(TA)-G

Commit message: Change an NPN LCSC part no. according to availability
Parts:
- Q901: LCSC C41095 -> C152538
Changed lines of the file:
@@
 F 2 "Package_TO_SOT_SMD:SOT-23" H 4000 4825 50  0001 L CIN
 F 3 "www.onsemi.com/pub/Collateral/MMBT5550LT1-D.PDF" H 3800 4900 50  0001 L CNN
-F 4 "C41095" H 3800 4900 50  0001 C CNN "LCSC"
+F 4 "C152538" H 3800 4900 50  0001 C CNN "LCSC"
 	1    3800 4900
 	1    0    0    -1

Commit message: Update parts according to JLC availability
Parts:
- Q901: LCSC C152538 -> C41095
Changed lines of the file:
@@
 F 2 "Package_TO_SOT_SMD:SOT-23" H 4000 4825 50  0001 L CIN
 F 3 "www.onsemi.com/pub/Collateral/MMBT5550LT1-D.PDF" H 3800 4900 50  0001 L CNN
-F 4 "C152538" H 3800 4900 50  0001 C CNN "LCSC"
+F 4 "C41095" H 3800 4900 50  0001 C CNN "LCSC"
 	1    3800 4900
 	1    0    0    -1
