File: ideal_diode.sch (KiCad schematic (older format))
At the start: 4 parts, among them Q1101 WST03P06, Q1102 BC857BS

Commit message: Add LCSC part number to Q1102
Parts:
- Q1102: LCSC (none) -> C8654
Changed lines of the file:
@@
 F 2 "Package_TO_SOT_SMD:SOT-363_SC-70-6" H 2550 2250 50  0001 C CNN
 F 3 "https://assets.nexperia.com/documents/data-sheet/BC857BS.pdf" H 2350 2150 50  0001 C CNN
+F 4 "C8654" H 2350 2150 50  0001 C CNN "LCSC"
 	1    2350 2150
 	-1   0    0    -1
@@
 F 2 "Package_TO_SOT_SMD:SOT-363_SC-70-6" H 3200 2250 50  0001 C CNN
 F 3 "https://assets.nexperia.com/documents/data-sheet/BC857BS.pdf" H 3000 2150 50  0001 C CNN
+F 4 "C8654" H 3000 2150 50  0001 C CNN "LCSC"
 	2    3000 2150
 	1    0    0    -1
