File: I2C.sch (KiCad schematic (older format))
At the start: 14 parts, among them J701 Conn_01x04, J702 Conn_01x04, U701 RCLAMP0524P-N

Commit message: Replace buck converter and CAN transceiver ICs
IC substitutions necessitated by component supply issues.
Other changes:
- Buck converter layout changes due to larger peripherals
- Isolated CAN transceiver replaced by separate digital isolators
  and transceivers. Layout changes.
- Changed JST XH conx to easier-to-use Phoenix MCs
- Removed dedicated Vin Prot conx (still available via VLink)
- Removed dedicated GND from left I/O header
Parts:
- J702: footprint Connector_PinHeader_2.54mm:PinHeader_1x04_P2.54mm_Vertical -> Connector_PinSocket_2.54mm:PinSocket_1x04_P2.54mm_Vertical; LCSC C358686 -> C124413
Changed lines of the file:
@@
 F 0 "J702" H 1568 3017 50  0000 C CNN
 F 1 "Conn_01x04" H 1568 2926 50  0000 C CNN
-F 2 "Connector_PinHeader_2.54mm:PinHeader_1x04_P2.54mm_Vertical" H 1650 2700 50  0001 C CNN
+F 2 "Connector_PinSocket_2.54mm:PinSocket_1x04_P2.54mm_Vertical" H 1650 2700 50  0001 C CNN
 F 3 "~" H 1650 2700 50  0001 C CNN
-F 4 "C358686" H 1650 2700 50  0001 C CNN "LCSC"
+F 4 "C124413" H 1650 2700 50  0001 C CNN "LCSC"
 	1    1650 2700
 	-1   0    0    -1
