File: canbus.sch (KiCad schematic (older format))
At the start: 16 parts, among them J601 Conn_01x04, J602 Conn_01x02, U602 ISO1050DUB, U603 H7550-H#

Commit message: Replace buck converter and CAN transceiver ICs
IC substitutions necessitated by component supply issues.
Other changes:
- Buck converter layout changes due to larger peripherals
- Isolated CAN transceiver replaced by separate digital isolators
  and transceivers. Layout changes.
- Changed JST XH conx to easier-to-use Phoenix MCs
- Removed dedicated Vin Prot conx (still available via VLink)
- Removed dedicated GND from left I/O header
Parts:
- removed J602: Conn_01x02, SH-ESP32:WireLink_1x02_P2.54mm, symbol Connector_Generic:Conn_01x02
- removed U602: ISO1050DUB, Package_SO:SOP-8_6.62x9.15mm_P2.54mm, symbol Interface_CAN_LIN:ISO1050DUB
- added C504: 100nF, Capacitor_SMD:C_0402_1005Metric, symbol Device:C
- added J501: Conn_01x02, Connector_PinHeader_2.54mm:PinHeader_1x02_P2.54mm_Vertical, symbol Connector_Generic:Conn_01x02
- added U501: SN65HVD231, Package_SO:SOIC-8_3.9x4.9mm_P1.27mm, symbol Interface_CAN_LIN:SN65HVD231
- added U502: ADuM1201AR, Package_SO:SOIC-8_3.9x4.9mm_P1.27mm, symbol Isolator:ADuM1201AR
- J601: footprint Connector_JST:JST_XH_B4B-XH-A_1x04_P2.50mm_Vertical -> Connector_Phoenix_MC:PhoenixContact_MCV_1,5_4-G-3.81_1x04_P3.81mm_Vertical; LCSC C8410 -> C8410
Connections:
- net labels added: D, R
- wire segments 53 -> 71
- no-connect marks 0 -> 1
Other:
- moved on the sheet: C602, C604
Changed lines of the file:
@@
 	2100 4800 2100 5000
 Wire Wire Line
-	6550 4000 6350 4000
-Wire Wire Line
-	6450 4300 6350 4300
-Wire Wire Line
-	6450 4350 6450 4300
+	7750 4200 7550 4200
+Wire Wire Line
+	7650 4600 7550 4600
+Wire Wire Line
+	7650 4650 7650 4600
 $Comp
 L power:GND #PWR0602
 U 1 1 5F3A993E
-P 6450 4350
-F 0 "#PWR0602" H 6450 4100 50  0001 C CNN
-F 1 "GND" H 6455 4177 50  0000 C CNN
-F 2 "" H 6450 4350 50  0001 C CNN
-F 3 "" H 6450 4350 50  0001 C CNN
-	1    6450 4350
-	-1   0    0    -1
-$EndComp
-$Comp
-L Interface_CAN_LIN:ISO1050DUB U602
-U 1 1 5F3944BA
-P 5950 4100
-F 0 "U602" H 5950 4467 50  0000 C CNN
-F 1 "ISO1050DUB" H 5950 4376 50  0000 C CNN
-F 2 "Package_SO:SOP-8_6.62x9.15mm_P2.54mm" H 5950 3750 50  0001 C CIN
-F 3 "http://www.ti.com/lit/ds/symlink/iso1050.pdf" H 5950 4050 50  0001 C CNN
-F 4 "C16428" H 5950 4100 50  0001 C CNN "LCSC"
-	1    5950 4100
+P 7650 4650
+F 0 "#PWR0602" H 7650 4400 50  0001 C CNN
+F 1 "GND" H 7655 4477 50  0000 C CNN
+F 2 "" H 7650 4650 50  0001 C CNN
+F 3 "" H 7650 4650 50  0001 C CNN
+	1    7650 4650
 	-1   0    0    -1
 $EndComp
@@
 L Device:C C?
 U 1 1 5F553562
-P 6800 3600
+P 8000 3800
 AR Path="/5D6F1C7C/5F553562" Ref="C?"  Part="1"
 AR Path="/5C348474/5F553562" Ref="C?"  Part="1"
 AR Path="/5F733BA4/5F553562" Ref="C604"  Part="1"
-F 0 "C604" H 6500 3650 50  0000 L CNN
-F 1 "100nF" H 6450 3550 50  0000 L CNN
-F 2 "Capacitor_SMD:C_0402_1005Metric" H 6838 3450 50  0001 C CNN
-F 3 "~" H 6800 3600 50  0001 C CNN
-F 4 "C1525" H 6800 3600 50  0001 C CNN "LCSC"
-	1    6800 3600
+F 0 "C604" H 7700 3850 50  0000 L CNN
+F 1 "100nF" H 7650 3750 50  0000 L CNN
+F 2 "Capacitor_SMD:C_0402_1005Metric" H 8038 3650 50  0001 C CNN
+F 3 "~" H 8000 3800 50  0001 C CNN
+F 4 "C1525" H 8000 3800 50  0001 C CNN "LCSC"
+	1    8000 3800
 	-1   0    0    -1
 $EndComp
@@
 L power:GND #PWR0603
 U 1 1 5F553DB4
-P 6800 3700
-F 0 "#PWR0603" H 6800 3450 50  0001 C CNN
-F 1 "GND" H 6805 3527 50  0000 C CNN
-F 2 "" H 6800 3700 50  0001 C CNN
-F 3 "" H 6800 3700 50  0001 C CNN
-	1    6800 3700
-	-1   0    0    -1
-$EndComp
-Wire Wire Line
-	6800 3450 6800 3350
-Wire Wire Line
-	6800 3350 6550 3350
-Wire Wire Line
-	6550 3350 6550 4000
-Wire Wire Line
-	6800 3750 6800 3700
+P 8000 3900
+F 0 "#PWR0603" H 8000 3650 50  0001 C CNN
+F 1 "GND" H 8005 3727 50  0000 C CNN
+F 2 "" H 8000 3900 50  0001 C CNN
+F 3 "" H 8000 3900 50  0001 C CNN
+	1    8000 3900
+	-1   0    0    -1
+$EndComp
+Wire Wire Line
+	8000 3650 8000 3550
+Wire Wire Line
+	8000 3550 7750 3550
+Wire Wire Line
+	7750 3550 7750 4200
+Wire Wire Line
+	8000 3950 8000 3900
 $Comp
 L Device:C C?
 U 1 1 5F55E792
-P 4900 4250
+P 5050 3750
 AR Path="/5D6F1C7C/5F55E792" Ref="C?"  Part="1"
 AR Path="/5C348474/5F55E792" Ref="C?"  Part="1"
 AR Path="/5F733BA4/5F55E792" Ref="C602"  Part="1"
-F 0 "C602" H 5015 4296 50  0000 L CNN
-F 1 "100nF" H 5015 4205 50  0000 L CNN
-F 2 "Capacitor_SMD:C_0402_1005Metric" H 4938 4100 50  0001 C CNN
-F 3 "~" H 4900 4250 50  0001 C CNN
-F 4 "C1525" H 4900 4250 50  0001 C CNN "LCSC"
-	1    4900 4250
-	-1   0    0    -1
-$EndComp
-Wire Wire Line
-	4900 4500 4900 4400
-Wire Wire Line
-	4650 4000 4900 4000
-Wire Wire Line
-	4900 4100 4900 4000
-Connection ~ 4900 4000
-Wire Wire Line
-	4900 4000 5550 4000
-Wire Wire Line
-	6350 4100 7100 4100
-Wire Wire Line
-	6350 4200 7100 4200
-Text HLabel 7100 4100 2    50   Input ~ 0
+F 0 "C602" H 5165 3796 50  0000 L CNN
+F 1 "100nF" H 5165 3705 50  0000 L CNN
+F 2 "Capacitor_SMD:C_0402_1005Metric" H 5088 3600 50  0001 C CNN
+F 3 "~" H 5050 3750 50  0001 C CNN
+F 4 "C1525" H 5050 3750 50  0001 C CNN "LCSC"
+	1    5050 3750
+	-1   0    0    -1
+$EndComp
+Wire Wire Line
+	5050 4000 5050 3900
+Wire Wire Line
+	4800 3500 5050 3500
+Wire Wire Line
+	5050 3600 5050 3500
+Wire Wire Line
+	7550 4500 8300 4500
+Wire Wire Line
+	7550 4300 8300 4300
+Text HLabel 8300 4500 2    50   Output ~ 0
 CAN_RX
-Text HLabel 7100 4200 2    50   Input ~ 0
+Text HLabel 8300 4300 2    50   Input ~ 0
 CAN_TX
-Text Label 4650 4000 2    50   ~ 0
+Text Label 4800 3500 2    50   ~ 0
 CAN_5V
 $Comp
@@
 Text Notes 1400 2050 2    50   ~ 0
 NMEA 2000
-Text Label 3050 2100 0    50   ~ 0
-CAN_GND
-Text Label 3050 2200 0    50   ~ 0
+Text Label 2250 2100 0    50   ~ 0
+CAN_GND
+Text Label 2250 2200 0    50   ~ 0
 CAN_12V
-Text Label 3050 2400 0    50   ~ 0
+Text Label 2250 2400 0    50   ~ 0
 CAN_L
-Text Label 3050 2300 0    50   ~ 0
+Text Label 2250 2300 0    50   ~ 0
 CAN_H
-Text Label 4900 4500 3    50   ~ 0
+Text Label 5050 4000 2    50   ~ 0
 CAN_GND
 Text Label 1950 4350 2    50   ~ 0
@@
 Text Label 1950 4150 2    50   ~ 0
 CAN_H
-Text Label 5550 4100 2    50   ~ 0
+Text Label 4900 4350 2    50   ~ 0
 CAN_H
-Text Label 5550 4200 2    50   ~ 0
+Text Label 4900 4450 2    50   ~ 0
 CAN_L
-Text Label 5550 4300 2    50   ~ 0
-CAN_GND
 Wire Wire Line
 	4600 1450 4850 1450
@@
 L power:+3.3V #PWR0103
 U 1 1 5F949C80
-P 6550 3350
-F 0 "#PWR0103" H 6550 3200 50  0001 C CNN
-F 1 "+3.3V" H 6565 3523 50  0000 C CNN
-F 2 "" H 6550 3350 50  0001 C CNN
-F 3 "" H 6550 3350 50  0001 C CNN
-	1    6550 3350
-	1    0    0    -1
-$EndComp
-Connection ~ 6550 3350
+P 7750 3550
+F 0 "#PWR0103" H 7750 3400 50  0001 C CNN
+F 1 "+3.3V" H 7765 3723 50  0000 C CNN
+F 2 "" H 7750 3550 50  0001 C CNN
+F 3 "" H 7750 3550 50  0001 C CNN
+	1    7750 3550
+	1    0    0    -1
+$EndComp
+Connection ~ 7750 3550
 $Comp
 L Connector_Generic:Conn_01x04 J601
@@
 F 0 "J601" H 1568 2517 50  0000 C CNN
 F 1 "Conn_01x04" H 1568 2426 50  0000 C CNN
-F 2 "Connector_JST:JST_XH_B4B-XH-A_1x04_P2.50mm_Vertical" H 1650 2200 50  0001 C CNN
+F 2 "Connector_Phoenix_MC:PhoenixContact_MCV_1,5_4-G-3.81_1x04_P3.81mm_Vertical" H 1650 2200 50  0001 C CNN
 F 3 "~" H 1650 2200 50  0001 C CNN
-F 4 "C8410" H 1650 2200 50  0001 C CNN "LCSC"
+F 4 " C8410" H 1650 2200 50  0001 C CNN "LCSC"
 	1    1650 2200
 	-1   0    0    -1
@@
 Text Notes 7250 1050 0    50   ~ 0
 Input voltage up to 40V
-$Comp
-L Connector_Generic:Conn_01x02 J?
-U 1 1 5FB62718
-P 8650 2500
-AR Path="/5F6FAF6E/5FB62718" Ref="J?"  Part="1"
-AR Path="/5F733BA4/5FB62718" Ref="J602"  Part="1"
-F 0 "J602" H 8568 2717 50  0000 C CNN
-F 1 "Conn_01x02" H 8568 2626 50  0000 C CNN
-F 2 "SH-ESP32:WireLink_1x02_P2.54mm" H 8650 2500 50  0001 C CNN
-F 3 "~" H 8650 2500 50  0001 C CNN
-	1    8650 2500
-	1    0    0    -1
-$EndComp
 Wire Wire Line
 	8450 2600 8300 2600
@@
 	8450 2500 8100 2500
 Wire Wire Line
-	1850 2200 3050 2200
-Wire Wire Line
-	1850 2100 3050 2100
+	1850 2200 2250 2200
+Wire Wire Line
+	1850 2100 2250 2100
 Text Label 8100 2500 2    50   ~ 0
 CAN12V_prot
@@
 	2100 4500 2200 4500
 Wire Wire Line
-	1850 2300 3050 2300
-Wire Wire Line
-	1850 2400 3050 2400
+	1850 2300 2250 2300
+Wire Wire Line
+	1850 2400 2250 2400
+$Comp
+L Isolator:ADuM1201AR U502
+U 1 1 6115AFFF
+P 7050 4400
+F 0 "U502" H 7050 4867 50  0000 C CNN
+F 1 "ADuM1201AR" H 7050 4776 50  0000 C CNN
+F 2 "Package_SO:SOIC-8_3.9x4.9mm_P1.27mm" H 7050 4000 50  0001 C CIN
+F 3 "https://www.analog.com/media/en/technical-documentation/data-sheets/ADuM1200_1201.pdf" H 7050 4300 50  0001 C CNN
+	1    7050 4400
+	1    0    0    -1
+$EndComp
+$Comp
+L Device:C C?
+U 1 1 6116F256
+P 6300 3800
+AR Path="/5D6F1C7C/6116F256" Ref="C?"  Part="1"
+AR Path="/5C348474/6116F256" Ref="C?"  Part="1"
+AR Path="/5F733BA4/6116F256" Ref="C504"  Part="1"
+F 0 "C504" H 6415 3846 50  0000 L CNN
+F 1 "100nF" H 6415 3755 50  0000 L CNN
+F 2 "Capacitor_SMD:C_0402_1005Metric" H 6338 3650 50  0001 C CNN
+F 3 "~" H 6300 3800 50  0001 C CNN
+F 4 "C1525" H 6300 3800 50  0001 C CNN "LCSC"
+	1    6300 3800
+	-1   0    0    -1
+$EndComp
+Wire Wire Line
+	6300 4050 6300 3950
+Wire Wire Line
+	6050 3550 6300 3550
+Wire Wire Line
+	6300 3650 6300 3550
+Connection ~ 6300 3550
+Text Label 6050 3550 2    50   ~ 0
+CAN_5V
+Text Label 6300 4050 2    50   ~ 0
+CAN_GND
+Wire Wire Line
+	6500 3550 6500 4200
+Wire Wire Line
+	6500 4200 6550 4200
+Wire Wire Line
+	6300 3550 6500 3550
+Wire Wire Line
+	5300 3500 5050 3500
+Wire Wire Line
+	5300 3500 5300 4050
+Connection ~ 5050 3500
+Wire Wire Line
+	6550 4300 6350 4300
+Wire Wire Line
+	6350 4300 6350 4250
+Wire Wire Line
+	6350 4250 5700 4250
+Wire Wire Line
+	5700 4350 6150 4350
+Wire Wire Line
+	6150 4350 6150 4500
+Wire Wire Line
+	6150 4500 6550 4500
+Wire Wire Line
+	5800 4550 5700 4550
+Wire Wire Line
+	5800 4600 5800 4550
+$Comp
+L Interface_CAN_LIN:SN65HVD231 U501
+U 1 1 6118CEF3
+P 5300 4350
+F 0 "U501" H 5200 4750 50  0000 C CNN
+F 1 "SN65HVD231" H 5000 4650 50  0000 C CNN
+F 2 "Package_SO:SOIC-8_3.9x4.9mm_P1.27mm" H 5300 3850 50  0001 C CNN
+F 3 "http://www.ti.com/lit/ds/symlink/sn65hvd230.pdf" H 5200 4750 50  0001 C CNN
+	1    5300 4350
+	-1   0    0    -1
+$EndComp
+Text Label 6500 4700 2    50   ~ 0
+CAN_GND
+Wire Wire Line
+	6500 4700 6550 4700
+Wire Wire Line
+	6550 4700 6550 4600
+NoConn ~ 5700 4450
+$Comp
+L Connector_Generic:Conn_01x02 J?
+U 1 1 611F3EE8
+P 8650 2600
+AR Path="/5F6FAF6E/611F3EE8" Ref="J?"  Part="1"
+AR Path="/5F733BA4/611F3EE8" Ref="J501"  Part="1"
+F 0 "J501" H 8568 2275 50  0000 C CNN
+F 1 "Conn_01x02" H 8568 2366 50  0000 C CNN
+F 2 "Connector_PinHeader_2.54mm:PinHeader_1x02_P2.54mm_Vertical" H 8650 2600 50  0001 C CNN
+F 3 "~" H 8650 2600 50  0001 C CNN
+	1    8650 2600
+	1    0    0    1
+$EndComp
+Wire Wire Line
+	5300 4900 5300 4750
+Text Label 5300 4900 3    50   ~ 0
+CAN_GND
+Text Label 5800 4600 3    50   ~ 0
+CAN_GND
+Text Label 6350 4250 0    50   ~ 0
+D
+Text Label 6150 4450 0    50   ~ 0
+R
 $EndSCHEMATC

Commit message: Change CAN Vcc to 3.3V; change components for availability
Parts:
- added R503: 10k, Resistor_SMD:R_0402_1005Metric, symbol Device:R_Small
- C603: value 2.2uF/50V -> 10uF/50V; footprint Capacitor_SMD:C_0805_2012Metric -> Capacitor_SMD:C_1206_3216Metric; LCSC C49217 -> C13585
- C605: value 2.2uF/16V -> 10uF/10V; LCSC C23630 -> C19702
- J501: LCSC (none) -> C492401
- U501: LCSC (none) -> C129257
- U502: LCSC (none) -> C9669
- U603: value H7550-H# -> PJ75AL33SA; LCSC C277875 -> C411736
Connections:
- net labels added: CAN_3V3
- net labels removed: CAN_5V
- wire segments 71 -> 72
Other:
- note added: "Input voltage up to 35V.\nOutput current at least 100mA."
- note added: "Rs provides slope control\nto limit EMI."
- note removed: "Input voltage up to 40V"
Changed lines of the file:
@@
 CAN_TX
 Text Label 4800 3500 2    50   ~ 0
-CAN_5V
+CAN_3V3
 $Comp
 L Device:Ferrite_Bead FB?
@@
 CAN_12V
 Text Label 7950 1450 0    50   ~ 0
-CAN_5V
+CAN_3V3
 Text Label 7000 2200 3    50   ~ 0
 CAN_GND
@@
 AR Path="/5F733BA4/5F94C99B" Ref="C605"  Part="1"
 F 0 "C605" H 7765 1846 50  0000 L CNN
-F 1 "2.2uF/16V" H 7765 1755 50  0000 L CNN
+F 1 "10uF/10V" H 7765 1755 50  0000 L CNN
 F 2 "Capacitor_SMD:C_0603_1608Metric" H 7688 1650 50  0001 C CNN
 F 3 "~" H 7650 1800 50  0001 C CNN
-F 4 "C23630" H 7650 1800 50  0001 C CNN "LCSC"
+F 4 "C19702" H 7650 1800 50  0001 C CNN "LCSC"
 	1    7650 1800
 	1    0    0    -1
@@
 AR Path="/5F733BA4/5F94C994" Ref="C603"  Part="1"
 F 0 "C603" H 6515 1846 50  0000 L CNN
-F 1 "2.2uF/50V" H 6515 1755 50  0000 L CNN
-F 2 "Capacitor_SMD:C_0805_2012Metric" H 6438 1650 50  0001 C CNN
+F 1 "10uF/50V" H 6515 1755 50  0000 L CNN
+F 2 "Capacitor_SMD:C_1206_3216Metric" H 6438 1650 50  0001 C CNN
 F 3 "~" H 6400 1800 50  0001 C CNN
-F 4 "C49217" H 6400 1800 50  0001 C CNN "LCSC"
+F 4 "C13585" H 6400 1800 50  0001 C CNN "LCSC"
 	1    6400 1800
 	1    0    0    -1
@@
 AR Path="/5F733BA4/5F94C95C" Ref="U603"  Part="1"
 F 0 "U603" H 7000 1917 50  0000 C CNN
-F 1 "H7550-H#" H 7000 1826 50  0000 C CNN
+F 1 "PJ75AL33SA" H 7000 1826 50  0000 C CNN
 F 2 "Package_TO_SOT_SMD:SOT-23" H 7000 1875 50  0001 C CIN
 F 3 "" H 7000 1650 50  0001 C CNN
-F 4 "C277875" H 7000 1550 50  0001 C CNN "LCSC"
+F 4 "C411736" H 7000 1550 50  0001 C CNN "LCSC"
 	1    7000 1550
 	1    0    0    -1
@@
 $EndComp
 Text Notes 7250 1050 0    50   ~ 0
-Input voltage up to 40V
+Input voltage up to 35V.\nOutput current at least 100mA.
 Wire Wire Line
 	8450 2600 8300 2600
@@
 F 2 "Package_SO:SOIC-8_3.9x4.9mm_P1.27mm" H 7050 4000 50  0001 C CIN
 F 3 "https://www.analog.com/media/en/technical-documentation/data-sheets/ADuM1200_1201.pdf" H 7050 4300 50  0001 C CNN
+F 4 "C9669" H 7050 4400 50  0001 C CNN "LCSC"
 	1    7050 4400
 	1    0    0    -1
@@
 Connection ~ 6300 3550
 Text Label 6050 3550 2    50   ~ 0
-CAN_5V
+CAN_3V3
 Text Label 6300 4050 2    50   ~ 0
 CAN_GND
@@
 Wire Wire Line
 	5800 4600 5800 4550
-$Comp
-L Interface_CAN_LIN:SN65HVD231 U501
-U 1 1 6118CEF3
-P 5300 4350
-F 0 "U501" H 5200 4750 50  0000 C CNN
-F 1 "SN65HVD231" H 5000 4650 50  0000 C CNN
-F 2 "Package_SO:SOIC-8_3.9x4.9mm_P1.27mm" H 5300 3850 50  0001 C CNN
-F 3 "http://www.ti.com/lit/ds/symlink/sn65hvd230.pdf" H 5200 4750 50  0001 C CNN
-	1    5300 4350
-	-1   0    0    -1
-$EndComp
 Text Label 6500 4700 2    50   ~ 0
 CAN_GND
@@
 F 2 "Connector_PinHeader_2.54mm:PinHeader_1x02_P2.54mm_Vertical" H 8650 2600 50  0001 C CNN
 F 3 "~" H 8650 2600 50  0001 C CNN
+F 4 "C492401" H 8650 2600 50  0001 C CNN "LCSC"
 	1    8650 2600
 	1    0    0    1
@@
 	5300 4900 5300 4750
 Text Label 5300 4900 3    50   ~ 0
-CAN_GND
-Text Label 5800 4600 3    50   ~ 0
 CAN_GND
 Text Label 6350 4250 0    50   ~ 0
@@
 Text Label 6150 4450 0    50   ~ 0
 R
+$Comp
+L Interface_CAN_LIN:SN65HVD231 U501
+U 1 1 6118CEF3
+P 5300 4350
+F 0 "U501" H 5200 4750 50  0000 C CNN
+F 1 "SN65HVD231" H 5000 4650 50  0000 C CNN
+F 2 "Package_SO:SOIC-8_3.9x4.9mm_P1.27mm" H 5300 3850 50  0001 C CNN
+F 3 "http://www.ti.com/lit/ds/symlink/sn65hvd230.pdf" H 5200 4750 50  0001 C CNN
+F 4 " C129257" H 5300 4350 50  0001 C CNN "LCSC"
+	1    5300 4350
+	-1   0    0    -1
+$EndComp
+$Comp
+L Device:R_Small R503
+U 1 1 611C6255
+P 5800 4700
+F 0 "R503" H 5859 4746 50  0000 L CNN
+F 1 "10k" H 5859 4655 50  0000 L CNN
+F 2 "Resistor_SMD:R_0402_1005Metric" H 5800 4700 50  0001 C CNN
+F 3 "~" H 5800 4700 50  0001 C CNN
+F 4 "C25744" H 5800 4700 50  0001 C CNN "LCSC"
+	1    5800 4700
+	1    0    0    -1
+$EndComp
+Wire Wire Line
+	5800 4900 5800 4800
+Text Notes 5700 5350 0    50   ~ 0
+Rs provides slope control\nto limit EMI.
+Text Label 5800 4900 0    50   ~ 0
+CAN_GND
 $EndSCHEMATC
