File: optocouplers.kicad_sch (KiCad schematic)
At the start: 21 parts, among them J901 Conn_01x04, Q901 MMBT5551L, U901 EL3H7(C)(TA)-G, U902 EL3H7(C)(TA)-G

Commit message: Change buck converter to LMR54410
Parts:
- Q901: footprint Package_TO_SOT_SMD:SOT-23 -> SH-ESP32:SOT-23
Changed lines of the file:
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@@
 	(title_block
 		(title "SH-ESP32")
-		(date "2024-06-27")
-		(rev "2.1.0")
+		(date "2024-09-24")
+		(rev "2.2.0")
 		(company "Hat Labs Oy")
 		(comment 1 "https://creativecommons.org/licenses/by-sa/4.0")
@@
 			)
 		)
-		(property "Description" ""
+		(property "Description" "Power symbol creates a global label with name \"GND\" , ground"
 			(at 54.61 129.54 0)
 			(effects
@@
 			)
 		)
-		(property "Footprint" "Package_TO_SOT_SMD:SOT-23"
+		(property "Footprint" "SH-ESP32:SOT-23"
 			(at 101.6 126.365 0)
 			(effects
@@
 			)
 		)
-		(property "Description" ""
+		(property "Description" "Power symbol creates a global label with name \"+3.3V\""
 			(at 72.39 53.34 0)
 			(effects
@@
 			)
 		)
-		(property "Description" ""
+		(property "Description" "Power symbol creates a global label with name \"GND\" , ground"
 			(at 72.39 74.93 0)
 			(effects
@@
 			)
 		)
-		(property "Description" ""
+		(property "Description" "Diode"
 			(at 107.95 111.76 0)
 			(effects
@@
 		)
 		(property "JLCPCB_CORRECTION" ""
+			(at 107.95 111.76 0)
+			(effects
+				(font
+					(size 1.27 1.27)
+				)
+				(hide yes)
+			)
+		)
+		(property "Sim.Device" "D"
+			(at 107.95 111.76 0)
+			(effects
+				(font
+					(size 1.27 1.27)
+				)
+				(hide yes)
+			)
+		)
+		(property "Sim.Pins" "1=K 2=A"
 			(at 107.95 111.76 0)
 			(effects
@@
 			)
 		)
-		(property "Description" ""
+		(property "Description" "Diode"
 			(at 104.14 63.5 0)
 			(effects
@@
 		)
 		(property "JLCPCB_CORRECTION" ""
+			(at 104.14 63.5 0)
+			(effects
+				(font
+					(size 1.27 1.27)
+				)
+				(hide yes)
+			)
+		)
+		(property "Sim.Device" "D"
+			(at 104.14 63.5 0)
+			(effects
+				(font
+					(size 1.27 1.27)
+				)
+				(hide yes)
+			)
+		)
+		(property "Sim.Pins" "1=K 2=A"
 			(at 104.14 63.5 0)
 			(effects
@@
 			)
 		)
-		(property "Description" ""
+		(property "Description" "AC/DC Optocoupler, Vce 70V, CTR 100-250%, SOP4"
 			(at 86.36 60.96 0)
 			(effects
@@
 			)
 		)
-		(property "Description" ""
+		(property "Description" "AC/DC Optocoupler, Vce 70V, CTR 100-250%, SOP4"
 			(at 66.04 127 0)
 			(effects
